File: 1001_macro_keypad/PCBs/architeuthis_dux.kicad_pcb (KiCad board)
At the start: 2 copper layers, 145.1 x 115 mm, 30 parts

Commit message: Schematic
Parts:
- removed MCU1: , ProMicro
- removed S1, S18, S7: , PG1350
- removed TRRS1: TRRS-PJ-320A-dual, TRRS-PJ-320A-dual
- added J1: ePaperModule, Connector_PinHeader_2.54mm:PinHeader_2x04_P2.54mm_Vertical, F.Cu at (156.0, 150.9)
- added J2: RotaryModule_01, Connector_PinHeader_2.54mm:PinHeader_1x05_P2.54mm_Vertical, F.Cu at (165.2, 151.5)
- added J3: RotaryModule_02, Connector_PinHeader_2.54mm:PinHeader_1x05_P2.54mm_Vertical, F.Cu at (169.8, 151.5)
- added SW01: MX_SW, Button_Switch_Keyboard:SW_Cherry_MX_1.00u_PCB, F.Cu at (206.2, 49.3)
- added SW10: MX_SW, Button_Switch_Keyboard:SW_Cherry_MX_1.00u_PCB, F.Cu at (229.1, 95.0)
- added SW11: MX_SW, Button_Switch_Keyboard:SW_Cherry_MX_1.00u_PCB, F.Cu at (252.0, 95.0)
- added SW12: MX_SW, Button_Switch_Keyboard:SW_Cherry_MX_1.00u_PCB, F.Cu at (274.6, 95.5)
- added SW13: MX_SW, Button_Switch_Keyboard:SW_Cherry_MX_1.00u_PCB, F.Cu at (192.0, 139.7)
- added SW14: MX_SW, Button_Switch_Keyboard:SW_Cherry_MX_1.00u_PCB, F.Cu at (214.9, 139.2)
- added SW2: MX_SW, Button_Switch_Keyboard:SW_Cherry_MX_1.00u_PCB, F.Cu at (229.1, 49.3)
- added SW3: MX_SW, Button_Switch_Keyboard:SW_Cherry_MX_1.00u_PCB, F.Cu at (252.0, 49.3)
- added SW4: MX_SW, Button_Switch_Keyboard:SW_Cherry_MX_1.00u_PCB, F.Cu at (274.1, 49.3)
- added SW5: MX_SW, Button_Switch_Keyboard:SW_Cherry_MX_1.00u_PCB, F.Cu at (206.2, 72.6)
- added SW6: MX_SW, Button_Switch_Keyboard:SW_Cherry_MX_1.00u_PCB, F.Cu at (229.1, 72.6)
- added SW7: MX_SW, Button_Switch_Keyboard:SW_Cherry_MX_1.00u_PCB, F.Cu at (252.0, 72.6)
- added SW8: MX_SW, Button_Switch_Keyboard:SW_Cherry_MX_1.00u_PCB, F.Cu at (274.3, 72.6)
- added SW9: MX_SW, Button_Switch_Keyboard:SW_Cherry_MX_1.00u_PCB, F.Cu at (206.2, 95.0)
- added U1: Pico, MCU_RaspberryPi_and_Boards:RPi_Pico_SMD_TH, F.Cu at (325.1, 127.5)
- moved S17 109.3 mm to (42.7, 53.3)
- moved S3 109.3 mm to (42.7, 53.3)
- moved S16 109.3 mm to (49.6, 72.1)
- moved S2 109.3 mm to (49.6, 72.1)
- moved S10 109.3 mm to (114.6, 77.0)
- moved S24 109.3 mm to (114.6, 77.0)
- moved S11 109.3 mm to (114.2, 57.0)
- moved S25 109.3 mm to (114.2, 57.0)
- moved S12 109.3 mm to (113.9, 37.0)
- moved S26 109.3 mm to (113.9, 37.0)
- moved S22 109.3 mm to (90.1, 50.3)
- moved S8 109.3 mm to (90.1, 50.3)
- moved S4 109.3 mm to (73.3, 77.4)
- moved S13 109.3 mm to (145.2, 111.5)
- moved S27 109.3 mm to (145.2, 111.5)
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Other:
- net class Default removed

Commit message: pcb modify
Parts:
- added D1: 1N4148, Diode_THT:D_DO-35_SOD27_P7.62mm_Horizontal, F.Cu at (208.3, 33.0)
Connections:
- SW01 pad 1: unconnected-(SW01-Pad1) -> Net-(D1-A)
- SW6 pad 1: unconnected-(SW6-Pad1) -> SW6

Commit message: 배션중
Parts:
- removed S10, S11, S12, S13, S14, S15, S16, S17, S19, S2, S20, S21, S22, S23, S24, S25, S26, S27, S28, S3, S4, S5, S6, S8, S9: , PG1350
- added D10: 1N4148, Diode_THT:D_DO-35_SOD27_P7.62mm_Horizontal, B.Cu at (173.4, 80.6)
- added D11: 1N4148, Diode_THT:D_DO-35_SOD27_P7.62mm_Horizontal, B.Cu at (194.4, 73.9)
- added D12: 1N4148, Diode_THT:D_DO-35_SOD27_P7.62mm_Horizontal, B.Cu at (217.9, 82.3)
- added D13: 1N4148, Diode_THT:D_DO-35_SOD27_P7.62mm_Horizontal, B.Cu at (254.0, 122.4)
- added D14: 1N4148, Diode_THT:D_DO-35_SOD27_P7.62mm_Horizontal, B.Cu at (274.2, 133.1)
- added D2: 1N4148, Diode_THT:D_DO-35_SOD27_P7.62mm_Horizontal, B.Cu at (162.7, 41.9)
- added D3: 1N4148, Diode_THT:D_DO-35_SOD27_P7.62mm_Horizontal, B.Cu at (188.3, 34.2)
- added D4: 1N4148, Diode_THT:D_DO-35_SOD27_P7.62mm_Horizontal, B.Cu at (217.5, 42.2)
- added D5: 1N4148, Diode_THT:D_DO-35_SOD27_P7.62mm_Horizontal, B.Cu at (147.1, 71.3)
- added D6: 1N4148, Diode_THT:D_DO-35_SOD27_P7.62mm_Horizontal, B.Cu at (167.8, 61.7)
- added D7: 1N4148, Diode_THT:D_DO-35_SOD27_P7.62mm_Horizontal, B.Cu at (191.0, 54.2)
- added D8: 1N4148, Diode_THT:D_DO-35_SOD27_P7.62mm_Horizontal, B.Cu at (217.5, 62.2)
- added D9: 1N4148, Diode_THT:D_DO-35_SOD27_P7.62mm_Horizontal, B.Cu at (154.8, 93.9)
- D1: moved to B.Cu
- moved U1 101.8 mm to (243.4, 66.7)
- moved D1 70.8 mm to (141.3, 55.8), turned to -70 degrees
- moved SW2 70.0 mm to (159.2, 50.9), turned to 15 degrees
- moved SW01 69.7 mm to (138.5, 65.4), turned to 20 degrees
- moved SW3 68.4 mm to (183.9, 42.9), turned to 10 degrees
- moved SW7 65.9 mm to (186.8, 62.7), turned to 10 degrees
- moved SW6 64.8 mm to (164.3, 70.2), turned to 15 degrees
- moved SW11 63.5 mm to (189.8, 82.4), turned to 10 degrees
- moved SW12 62.7 mm to (212.2, 89.7), turned to 0.45 degrees
- moved SW4 62.6 mm to (211.5, 49.7), turned to 0.45 degrees
- moved SW8 62.6 mm to (211.8, 69.7), turned to 0.45 degrees
- moved SW5 62.0 mm to (145.3, 84.2), turned to 20 degrees
- moved SW10 59.8 mm to (169.5, 89.6), turned to 15 degrees
- moved SW9 54.7 mm to (152.1, 103.0), turned to 20 degrees
- moved SW13 54.7 mm to (245.0, 126.0), turned to -29.25 degrees
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Connections:
- D1 pad 1: unconnected-(D1-K-Pad1) -> ROW0
- SW01 pad 2: GND -> COL0
- SW10 pad 1: unconnected-(SW10-Pad1) -> Net-(D10-A)
- SW10 pad 2: GND -> COL1
- SW11 pad 1: unconnected-(SW11-Pad1) -> Net-(D11-A)
- SW11 pad 2: GND -> COL2
- SW12 pad 1: unconnected-(SW12-Pad1) -> Net-(D12-A)
- SW12 pad 2: GND -> COL3
- SW13 pad 1: unconnected-(SW13-Pad1) -> Net-(D13-A)
- SW13 pad 2: GND -> COL2
- SW14 pad 1: unconnected-(SW14-Pad1) -> Net-(D14-A)
- SW14 pad 2: GND -> COL3
- SW2 pad 1: unconnected-(SW2-Pad1) -> Net-(D2-A)
- SW2 pad 2: GND -> COL1
- SW3 pad 1: unconnected-(SW3-Pad1) -> Net-(D3-A)
- SW3 pad 2: GND -> COL2
- SW4 pad 1: unconnected-(SW4-Pad1) -> Net-(D4-A)
- SW4 pad 2: GND -> COL3
- SW5 pad 1: unconnected-(SW5-Pad1) -> Net-(D5-A)
- SW5 pad 2: GND -> COL0
- SW6 pad 1: SW6 -> Net-(D6-A)
- SW6 pad 2: GND -> COL1
- SW7 pad 1: unconnected-(SW7-Pad1) -> Net-(D7-A)
- SW7 pad 2: GND -> COL2
- SW8 pad 1: unconnected-(SW8-Pad1) -> Net-(D8-A)
- SW8 pad 2: GND -> COL3
- SW9 pad 1: unconnected-(SW9-Pad1) -> Net-(D9-A)
- SW9 pad 2: GND -> COL0
- U1 pad 1: unconnected-(U1-GPIO0-Pad1) -> ROW0
- U1 pad 10: unconnected-(U1-GPIO7-Pad10) -> COL2
- U1 pad 2: unconnected-(U1-GPIO1-Pad2) -> ROW1
- U1 pad 4: unconnected-(U1-GPIO2-Pad4) -> ROW2
- U1 pad 5: unconnected-(U1-GPIO3-Pad5) -> ROW3
- U1 pad 6: unconnected-(U1-GPIO4-Pad6) -> COL1
- U1 pad 7: unconnected-(U1-GPIO5-Pad7) -> COL0
- U1 pad 9: unconnected-(U1-GPIO6-Pad9) -> COL3
Routing:
- net COL1: track 0.00 -> 258.9 mm
- net COL0: track 0.00 -> 213.2 mm
- net COL3: track 0.00 -> 193.7 mm
- net COL2: track 0.00 -> 174.6 mm
- net ROW2: track 0.00 -> 116.4 mm
- net ROW0: track 0.00 -> 107.5 mm
- net ROW1: track 0.00 -> 106.0 mm
- net ROW3: track 0.00 -> 102.4 mm
- net Net-(D14-A): track 0.00 -> 9.58 mm
- net Net-(D5-A): track 0.00 -> 7.55 mm
- net Net-(D13-A): track 0.00 -> 6.55 mm
- net Net-(D10-A): track 0.00 -> 6.54 mm
- net Net-(D11-A): track 0.00 -> 6.44 mm
- net Net-(D1-A): track 0.00 -> 6.40 mm
- net Net-(D2-A): track 0.00 -> 6.22 mm
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Other:
- board outline removed

Commit message: 재배선
Parts:
- moved D1 15.3 mm to (146.3, 70.3), turned to 110 degrees
- moved D3 15.3 mm to (190.9, 49.2), turned to 100 degrees
- moved D2 15.3 mm to (166.7, 56.7), turned to 105 degrees
- moved D5 4.97 mm to (148.5, 76.1)
- moved D14 4.85 mm to (269.9, 135.3)
- moved SW01 0.07 mm to (138.4, 65.5)
Connections:
- SW01 pad 2: COL0 -> COL2
- SW10 pad 2: COL1 -> COL3
- SW11 pad 2: COL2 -> COL1
- SW12 pad 2: COL3 -> COL0
- SW13 pad 2: COL2 -> COL3
- SW14 pad 2: COL3 -> COL2
- SW2 pad 2: COL1 -> COL3
- SW3 pad 2: COL2 -> COL1
- SW4 pad 2: COL3 -> COL0
- SW5 pad 2: COL0 -> COL2
- SW6 pad 2: COL1 -> COL3
- SW7 pad 2: COL2 -> COL1
- SW8 pad 2: COL3 -> COL0
- SW9 pad 2: COL0 -> COL2
- U1 pad 10: COL2 -> COL3
- U1 pad 6: COL1 -> COL0
- U1 pad 7: COL0 -> COL1
- U1 pad 9: COL3 -> COL2
Routing:
- net COL1: track 258.9 -> 128.1 mm
- net COL0: track 213.2 -> 103.0 mm
- net COL2: track 174.6 -> 245.9 mm
- net ROW0: track 107.5 -> 100.6 mm
- net ROW3: track 102.4 -> 98.9 mm
- net Net-(D14-A): track 9.58 -> 6.15 mm
- net Net-(D5-A): track 7.55 -> 6.20 mm
- net COL3: track 193.7 -> 192.8 mm
- net ROW1: track 106.0 -> 106.6 mm
Other:
- board outline added: 150.7 x 127.4 mm

Commit message: ePaper
Parts:
- moved J2 119.1 mm to (265.2, 86.9)
- moved J3 103.8 mm to (264.2, 108.2)
- moved J1 95.9 mm to (241.0, 106.5), turned to -90 degrees
- moved U1 9.43 mm to (234.1, 65.7)
- moved D7 1.58 mm to (191.4, 55.7)
Connections:
- J1 pad 7: unconnected-(J1-Pin_7-Pad7) -> GND
- J1 pad 8: unconnected-(J1-Pin_8-Pad8) -> +5V
- J2 pad 1: unconnected-(J2-Pin_1-Pad1) -> +5V
- J2 pad 5: unconnected-(J2-Pin_5-Pad5) -> GND
- J3 pad 1: unconnected-(J3-Pin_1-Pad1) -> +5V
- J3 pad 5: unconnected-(J3-Pin_5-Pad5) -> GND
- U1 pad 40: unconnected-(U1-VBUS-Pad40) -> +5V
Routing:
- net ROW3: track 98.9 -> 27.3 mm
- net ROW0: track 100.6 -> 90.8 mm
- net COL2: track 245.9 -> 252.2 mm
- net COL3: track 192.8 -> 196.5 mm
- net ROW2: track 116.5 -> 113.6 mm
- net COL1: track 128.1 -> 125.2 mm
- net ROW1: track 106.6 -> 104.8 mm
- net (no net): vias 0 -> 1
- added copper zone on F.Cu, net GND
Other:
- board size 150.7 x 127.4 mm -> 149.4 x 116.8 mm

Commit message: 일부수정
Parts:
- moved J1 44.8 mm to (265.9, 69.3)
Connections:
- J1 pad 1: unconnected-(J1-BUSY-Pad1) -> +5V
- J1 pad 2: unconnected-(J1-RES-Pad2) -> GND
- J1 pad 7: GND -> unconnected-(J1-GND-Pad7)
- J1 pad 8: +5V -> unconnected-(J1-VCC-Pad8)
Routing:
- net ROW3: track 27.3 -> 108.0 mm

Commit message: e페이퍼모듈 풋프린트 추가
Parts:
- added REF**: e-Paper Module 2.13, ePaper:e-Paper Module 2.13, F.Cu at (327.1, 85.0)
- moved J3 4.29 mm to (265.0, 104.0)
- moved J2 0.44 mm to (265.0, 86.5)
Other:
- outline, holes or cut-outs redrawn

Commit message: 배선작업 거의 완료
Parts:
- added REF**: MountingHole_2.1mm, MountingHole:MountingHole_2.1mm, F.Cu at (196.0, 50.0)
- added REF**: MountingHole_2.1mm, MountingHole:MountingHole_2.1mm, F.Cu at (197.0, 102.0)
- added REF**: MountingHole_2.1mm, MountingHole:MountingHole_2.1mm, F.Cu at (259.0, 120.0)
- added REF**: MountingHole_2.1mm, MountingHole:MountingHole_2.1mm, F.Cu at (258.0, 40.0)
- added REF**: MountingHole_2.1mm, MountingHole:MountingHole_2.1mm, F.Cu at (242.0, 101.0)
- added REF**: MountingHole_2.1mm, MountingHole:MountingHole_2.1mm, F.Cu at (225.0, 116.0)
- added REF**: MountingHole_2.1mm, MountingHole:MountingHole_2.1mm, F.Cu at (248.0, 151.0)
- added REF**: MountingHole_2.1mm, MountingHole:MountingHole_2.1mm, F.Cu at (171.0, 58.0)
- added REF**: MountingHole_2.1mm, MountingHole:MountingHole_2.1mm, F.Cu at (167.0, 110.0)
- added REF**: MountingHole_2.1mm, MountingHole:MountingHole_2.1mm, F.Cu at (144.0, 55.0)
- moved J1 29.4 mm to (251.0, 44.0), turned to 0 degrees
- moved J2 17.9 mm to (254.0, 72.4)
- moved J3 17.9 mm to (254.0, 89.9)
Connections:
- J1 pad 3: unconnected-(J1-D/C-Pad3) -> Net-(J1-D/C)
- J1 pad 4: unconnected-(J1-CS-Pad4) -> Net-(J1-CS)
- J1 pad 5: unconnected-(J1-SCL-Pad5) -> Net-(J1-SCL)
- J1 pad 6: unconnected-(J1-SDA-Pad6) -> Net-(J1-SDA)
- J1 pad 7: unconnected-(J1-GND-Pad7) -> Net-(J1-GND)
- J1 pad 8: unconnected-(J1-VCC-Pad8) -> Net-(J1-VCC)
- J2 pad 2: unconnected-(J2-KEY-Pad2) -> Net-(J2-KEY)
- J2 pad 3: unconnected-(J2-S2-Pad3) -> Net-(J2-S2)
- J2 pad 4: unconnected-(J2-S1-Pad4) -> Net-(J2-S1)
- J3 pad 2: unconnected-(J3-Pin_2-Pad2) -> Net-(J3-Pin_2)
- J3 pad 3: unconnected-(J3-Pin_3-Pad3) -> Net-(J3-Pin_3)
- J3 pad 4: unconnected-(J3-Pin_4-Pad4) -> Net-(J3-Pin_4)
- U1 pad 19: unconnected-(U1-GPIO14-Pad19) -> Net-(J3-Pin_3)
- U1 pad 20: unconnected-(U1-GPIO15-Pad20) -> Net-(J3-Pin_4)
- U1 pad 21: unconnected-(U1-GPIO16-Pad21) -> Net-(J3-Pin_2)
- U1 pad 22: unconnected-(U1-GPIO17-Pad22) -> Net-(J2-S1)
- U1 pad 24: unconnected-(U1-GPIO18-Pad24) -> Net-(J2-S2)
- U1 pad 25: unconnected-(U1-GPIO19-Pad25) -> Net-(J2-KEY)
- U1 pad 26: unconnected-(U1-GPIO20-Pad26) -> Net-(J1-CS)
- U1 pad 27: unconnected-(U1-GPIO21-Pad27) -> Net-(J1-SDA)
- U1 pad 29: unconnected-(U1-GPIO22-Pad29) -> Net-(J1-VCC)
- U1 pad 31: unconnected-(U1-GPIO26_ADC0-Pad31) -> Net-(J1-GND)
- U1 pad 32: unconnected-(U1-GPIO27_ADC1-Pad32) -> Net-(J1-SCL)
- U1 pad 34: unconnected-(U1-GPIO28_ADC2-Pad34) -> Net-(J1-D/C)
Routing:
- net +5V: track 0.00 -> 70.0 mm
- net Net-(J1-CS): track 0.00 -> 37.2 mm
- net Net-(J3-Pin_4): track 0.00 -> 32.3 mm
- net Net-(J3-Pin_3): track 0.00 -> 32.0 mm
- net Net-(J1-SDA): track 0.00 -> 31.8 mm
- net Net-(J1-VCC): track 0.00 -> 23.2 mm
- net Net-(J1-SCL): track 0.00 -> 17.1 mm
- net Net-(J1-GND): track 0.00 -> 17.1 mm
- net Net-(J1-D/C): track 0.00 -> 16.2 mm
- net Net-(J2-S1): track 0.00 -> 14.0 mm
- net Net-(J2-KEY): track 0.00 -> 13.0 mm
- net Net-(J2-S2): track 0.00 -> 13.0 mm
- net Net-(J3-Pin_2): track 0.00 -> 12.1 mm
- net ROW2: track 113.6 -> 112.0 mm
- net ROW3: track 108.0 -> 109.3 mm
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- added copper zone on B.Cu, net GND
Other:
- board size 149.4 x 116.8 mm -> 145.7 x 117.9 mm
