File: 1003_pedal/000_electra_distortion/kicadProj/electra_000/electra_000.kicad_pcb (KiCad board)
At the start: 2 copper layers, 17 parts, among them J1 AudioJack2, J2 AudioJack2, Q1 Q_NPN_BCE, SW1 SW_Slide_DPDT

Commit message: veroboard start
Routing:
- net (no net): track 0.00 -> 58.5 mm
- net Net-(J2-PadT): track 0.00 -> 49.9 mm
Changed lines of the file:
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@@
+		)
+	)
+	(gr_rect
+		(start 195.5 50)
+		(end 220.5 114)
+		(stroke
+			(width 0.2)
+			(type default)
+		)
+		(fill no)
+		(layer "F.Cu")
+	)
+	(segment
+		(start 218.5 53)
+		(end 218.5 111.5)
+		(width 1.5)
+		(layer "F.Cu")
+		(net "")
+	)
+	(segment
+		(start 150 56.5)
+		(end 164.5 71)
+		(width 0.2)
+		(layer "F.Cu")
+		(net "Net-(J2-PadT)")
+	)
+	(segment
+		(start 149.96205 56.53795)
+		(end 150 56.5)
+		(width 0.2)
+		(layer "F.Cu")
+		(net "Net-(J2-PadT)")
+	)
+	(segment
+		(start 164.5 71)
+		(end 164.5 73.5)
+		(width 0.2)
+		(layer "F.Cu")
+		(net "Net-(J2-PadT)")
+	)
+	(segment
+		(start 123.08 56.53795)
+		(end 149.96205 56.53795)
+		(width 0.2)
+		(layer "F.Cu")
+		(net "Net-(J2-PadT)")
+	)
+	(zone
+		(layer "B.Cu")
+		(hatch edge 0.5)
+		(connect_pads
+			(clearance 0)
+		)
+		(min_thickness 0.25)
+		(keepout
+			(tracks not_allowed)
+			(vias not_allowed)
+			(pads not_allowed)
+			(copperpour allowed)
+			(footprints allowed)
+		)
+		(placement
+			(enabled no)
+			(sheetname "/")
+		)
+		(fill
+			(thermal_gap 0.5)
+			(thermal_bridge_width 0.5)
+			(island_removal_mode 0)
+		)
+		(polygon
+			(pts
+				(xy 195.5 50) (xy 220.5 50) (xy 220.5 114) (xy 195.5 114)
+			)
 		)
 	)

Commit message: schematic
Parts:
- added REF**: VeroBoard_25x64, VeroBoard:Veroboard_25x64, F.Cu at (202.5, 72.0)
- R2: footprint Resistor_THT:R_Axial_DIN0207_L6.3mm_D2.5mm_P7.62mm_Horizontal -> Resistor_THT:R_Axial_DIN0207_L6.3mm_D2.5mm_P2.54mm_Vertical
- moved R2 110.4 mm to (195.0, 47.0), turned to 180 degrees
- moved R1 99.9 mm to (192.5, 44.5), turned to 0 degrees
Routing:
- net (no net): track 58.5 -> 0.00 mm

Commit message: layout
Parts:
- added ?: , Monkey_Riot_Pedals_Library:1590B, F.Cu at (86.4, 95.1)
- D1, D2: footprint Diode_THT:D_DO-41_SOD81_P10.16mm_Horizontal -> Diode_THT:D_DO-41_SOD81_P7.62mm_Horizontal
- Q1: value Q_NPN_BCE -> Q_NPN_CBE; footprint Package_TO_SOT_THT:TO-92_Inline -> Monkey_Riot_Pedals_Library:TO-92L_INLINE_WIDE
- R1: footprint Resistor_THT:R_Axial_DIN0207_L6.3mm_D2.5mm_P7.62mm_Horizontal -> Resistor_THT:R_Axial_DIN0204_L3.6mm_D1.6mm_P7.62mm_Horizontal
- R2: footprint Resistor_THT:R_Axial_DIN0207_L6.3mm_D2.5mm_P2.54mm_Vertical -> Resistor_THT:R_Axial_DIN0204_L3.6mm_D1.6mm_P2.54mm_Vertical
- R3: footprint Resistor_THT:R_Axial_DIN0207_L6.3mm_D2.5mm_P7.62mm_Horizontal -> Resistor_THT:R_Axial_DIN0309_L9.0mm_D3.2mm_P12.70mm_Horizontal
- moved Q1 121.6 mm to (213.4, 71.1), turned to 180 degrees
- moved C3 115.7 mm to (221.1, 68.6)
- moved R3 113.5 mm to (208.3, 81.3)
- moved C1 112.4 mm to (213.4, 63.5), turned to 0 degrees
- moved D3 106.0 mm to (221.0, 94.0), turned to 180 degrees
- moved D1 106.0 mm to (221.0, 99.1), turned to 180 degrees
- moved C2 100.2 mm to (210.8, 86.4), turned to 180 degrees
- moved D2 98.6 mm to (213.4, 104.1)
- moved D4 97.5 mm to (213.4, 91.4)
- moved SW1 91.3 mm to (233.8, 101.6)
- moved REF** 58.3 mm to (256.5, 94.0)
- moved J2 44.9 mm to (129.0, 108.1)
- moved R2 28.3 mm to (213.4, 68.6)
- moved R1 25.3 mm to (205.7, 66.0)
- moved RV1 24.1 mm to (104.1, 76.2)
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Connections:
- Q1 pad 1: Net-(Q1-B) -> Net-(Q1-C)
- Q1 pad 2: Net-(Q1-C) -> Net-(Q1-B)
- R2 pad 1: Net-(Q1-B) -> Net-(Q1-C)
- R2 pad 2: Net-(Q1-C) -> Net-(Q1-B)
Routing:
- net Net-(J2-PadT): track 49.9 -> 0.00 mm
Other:
- board outline added: 25.4 x 66 mm

Commit message: pcb update
Parts:
- R3: footprint Resistor_THT:R_Axial_DIN0309_L9.0mm_D3.2mm_P12.70mm_Horizontal -> Resistor_THT:R_Axial_DIN0207_L6.3mm_D2.5mm_P10.16mm_Horizontal
- moved R1 17.8 mm to (223.5, 66.0), turned to 180 degrees
- moved D1 12.8 mm to (208.3, 100.6), turned to 0 degrees
- moved C3 12.8 mm to (208.3, 68.6), turned to 180 degrees
- moved D3 12.7 mm to (208.3, 94.0), turned to 0 degrees
- moved R3 12.7 mm to (221.0, 81.3), turned to 180 degrees
- moved C2 7.66 mm to (218.5, 86.4), turned to 0 degrees
- moved D2 2.54 mm to (215.9, 104.1), turned to 180 degrees
- moved D4 2.54 mm to (215.9, 91.4), turned to 180 degrees
- moved Q1 2.54 mm to (215.9, 71.1), turned to 0 degrees
- moved R2 2.54 mm to (215.9, 68.6), turned to 0 degrees
- moved C1 2.50 mm to (215.9, 63.5), turned to 180 degrees
- moved SW1 2.16 mm to (231.6, 101.6)
Routing:
- net Net-(D3-A): vias 0 -> 1
- net Net-(D1-A): vias 0 -> 1
- net GND: vias 0 -> 2

Commit message: almost finished and 3d models
Parts:
- removed the REF** at (256.5, 94.0)
- added >NAME: >VALUE, 3pdt:STOMP-SWITCH-3PDT, F.Cu at (86.6, 120.9)
- added REF**: wire_pad_round, Monkey_Riot_Pedals_Library:wire_pad_round, F.Cu at (205.7, 65.8)
- moved C1 2.58 mm to (213.3, 63.5)
- moved C3 2.56 mm to (205.7, 68.4), turned to -120 degrees
- moved Q1 1.78 mm to (215.9, 72.9)
- moved D4 0.25 mm to (215.9, 91.2)
Routing:
- net Net-(D1-K): vias 0 -> 1
- net +9VA: vias 0 -> 1
Other:
- board size 25.4 x 66 mm -> 25.7 x 65.5 mm
