File: 1003_pedal/000_electra_distortion/kicadProj/electra_000/electra_000.kicad_sch (KiCad schematic)
At the start: 17 parts, among them J1 AudioJack2, J2 AudioJack2, Q1 Q_NPN_BCE, SW1 SW_Slide_DPDT

Commit message: library added
Parts:
- RV1, RV2, RV3: footprint Potentiometer_THT:Potentiometer_Alps_RK09L_Single_Vertical -> Monkey_Riot_Pedals_Library:POT_16MM
- SW1: footprint Button_Switch_THT:SW_DIP_SPSTx04_Slide_6.7x11.72mm_W7.62mm_P2.54mm_LowProfile -> Monkey_Riot_Pedals_Library:DPDT.LUGS
Changed lines of the file:
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@@
 			)
 		)
-		(property "Footprint" "Potentiometer_THT:Potentiometer_Alps_RK09L_Single_Vertical"
+		(property "Footprint" "Monkey_Riot_Pedals_Library:POT_16MM"
 			(at 173.99 66.04 0)
 			(hide yes)
@@
 			)
 		)
-		(property "Footprint" "Potentiometer_THT:Potentiometer_Alps_RK09L_Single_Vertical"
+		(property "Footprint" "Monkey_Riot_Pedals_Library:POT_16MM"
 			(at 153.67 48.26 0)
 			(hide yes)
@@
 			)
 		)
-		(property "Footprint" "Potentiometer_THT:Potentiometer_Alps_RK09L_Single_Vertical"
+		(property "Footprint" "Monkey_Riot_Pedals_Library:POT_16MM"
 			(at 111.76 44.45 0)
 			(hide yes)
@@
 			)
 		)
-		(property "Footprint" "Button_Switch_THT:SW_DIP_SPSTx04_Slide_6.7x11.72mm_W7.62mm_P2.54mm_LowProfile"
+		(property "Footprint" "Monkey_Riot_Pedals_Library:DPDT.LUGS"
 			(at 182.88 102.87 0)
 			(hide yes)
