File: 1003_pedal/000_electra_distortion/kicadProj/electra_000/electra_000.kicad_sch (KiCad schematic)
At the start: 17 parts, among them J1 AudioJack2, J2 AudioJack2, Q1 Q_NPN_BCE, SW1 SW_Slide_DPDT

Commit message: schematic
Parts:
- C1, C2, C3: KiLib_Generator (none) -> capacitor/THT/other
- D1, D2, D3, D4: KiLib_Generator (none) -> diode/THT
- R1, R3: KiLib_Generator (none) -> resistor/THT
- R2: footprint Resistor_THT:R_Axial_DIN0207_L6.3mm_D2.5mm_P7.62mm_Horizontal -> Resistor_THT:R_Axial_DIN0207_L6.3mm_D2.5mm_P2.54mm_Vertical; KiLib_Generator (none) -> resistor/THT
Changed lines of the file:
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@@
+			)
+		)
+		(property "KiLib_Generator" "capacitor/THT/other"
+			(at 163.83 44.45 0)
+			(hide yes)
+			(show_name no)
+			(do_not_autoplace no)
+			(effects
+				(font
+					(size 1.27 1.27)
+				)
 			)
 		)
@@
 			)
 		)
+		(property "KiLib_Generator" "resistor/THT"
+			(at 129.54 110.49 0)
+			(hide yes)
+			(show_name no)
+			(do_not_autoplace no)
+			(effects
+				(font
+					(size 1.27 1.27)
+				)
+			)
+		)
 		(pin "2"
 		)
@@
 			)
 		)
+		(property "KiLib_Generator" "diode/THT"
+			(at 152.4 83.82 0)
+			(hide yes)
+			(show_name no)
+			(do_not_autoplace no)
+			(effects
+				(font
+					(size 1.27 1.27)
+				)
+			)
+		)
 		(pin "1"
 		)
@@
 			)
 		)
+		(property "KiLib_Generator" "resistor/THT"
+			(at 129.54 58.42 0)
+			(hide yes)
+			(show_name no)
+			(do_not_autoplace no)
+			(effects
+				(font
+					(size 1.27 1.27)
+				)
+			)
+		)
 		(pin "1"
 		)
@@
 			)
 		)
+		(property "KiLib_Generator" "capacitor/THT/other"
+			(at 163.83 66.04 0)
+			(hide yes)
+			(show_name no)
+			(do_not_autoplace no)
+			(effects
+				(font
+					(size 1.27 1.27)
+				)
+			)
+		)
 		(pin "1"
 		)
@@
 			)
 		)
+		(property "KiLib_Generator" "diode/THT"
+			(at 152.4 97.79 0)
+			(hide yes)
+			(show_name no)
+			(do_not_autoplace no)
+			(effects
+				(font
+					(size 1.27 1.27)
+				)
+			)
+		)
 		(pin "1"
 		)
@@
 			)
 		)
+		(property "KiLib_Generator" "capacitor/THT/other"
+			(at 143.51 62.23 0)
+			(hide yes)
+			(show_name no)
+			(do_not_autoplace no)
+			(effects
+				(font
+					(size 1.27 1.27)
+				)
+			)
+		)
 		(pin "1"
 		)
@@
 			)
 		)
-		(property "Footprint" "Resistor_THT:R_Axial_DIN0207_L6.3mm_D2.5mm_P7.62mm_Horizontal"
+		(property "Footprint" "Resistor_THT:R_Axial_DIN0207_L6.3mm_D2.5mm_P2.54mm_Vertical"
 			(at 125.73 64.008 90)
 			(hide yes)
@@
 			)
 		)
+		(property "KiLib_Generator" "resistor/THT"
+			(at 125.73 62.23 0)
+			(hide yes)
+			(show_name no)
+			(do_not_autoplace no)
+			(effects
+				(font
+					(size 1.27 1.27)
+				)
+			)
+		)
 		(pin "2"
 		)
@@
 			)
 		)
+		(property "KiLib_Generator" "diode/THT"
+			(at 152.4 78.74 0)
+			(hide yes)
+			(show_name no)
+			(do_not_autoplace no)
+			(effects
+				(font
+					(size 1.27 1.27)
+				)
+			)
+		)
 		(pin "1"
 		)
@@
 			(at 152.4 106.68 0)
 			(hide yes)
+			(show_name no)
+			(do_not_autoplace no)
+			(effects
+				(font
+					(size 1.27 1.27)
+				)
+			)
+		)
+		(property "KiLib_Generator" "diode/THT"
+			(at 152.4 106.68 0)
+			(hide yes)

Commit message: layout
Parts:
- D1, D2: footprint Diode_THT:D_DO-41_SOD81_P10.16mm_Horizontal -> Diode_THT:D_DO-41_SOD81_P7.62mm_Horizontal
- Q1: value Q_NPN_BCE -> Q_NPN_CBE; footprint Package_TO_SOT_THT:TO-92_Inline -> Monkey_Riot_Pedals_Library:TO-92L_INLINE_WIDE
- R1: footprint Resistor_THT:R_Axial_DIN0207_L6.3mm_D2.5mm_P7.62mm_Horizontal -> Resistor_THT:R_Axial_DIN0204_L3.6mm_D1.6mm_P7.62mm_Horizontal
- R2: footprint Resistor_THT:R_Axial_DIN0207_L6.3mm_D2.5mm_P2.54mm_Vertical -> Resistor_THT:R_Axial_DIN0204_L3.6mm_D1.6mm_P2.54mm_Vertical
- R3: footprint Resistor_THT:R_Axial_DIN0207_L6.3mm_D2.5mm_P7.62mm_Horizontal -> Resistor_THT:R_Axial_DIN0309_L9.0mm_D3.2mm_P12.70mm_Horizontal
Connections:
- net at C2.1, Q1.1 (B): now also R2.2; no longer R2.1
- net at C1.1, Q1.2 (C), R1.2: now also R2.1; no longer R2.2
Other:
- moved on the sheet: R2
Changed lines of the file:
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@@
+	(wire
+		(pts
+			(xy 121.92 66.04) (xy 160.02 66.04)
+		)
+		(stroke
+			(width 0)
+			(type default)
+		)
+	)
 	(wire
 		(pts
@@
 		(pts
 			(xy 148.59 62.23) (xy 148.59 78.74)
-		)
-		(stroke
-			(width 0)
-			(type default)
-		)
-	)
-	(wire
-		(pts
-			(xy 160.02 66.04) (xy 121.92 66.04)
 		)
 		(stroke
@@
 			)
 		)
-		(property "Footprint" "Resistor_THT:R_Axial_DIN0207_L6.3mm_D2.5mm_P7.62mm_Horizontal"
+		(property "Footprint" "Resistor_THT:R_Axial_DIN0309_L9.0mm_D3.2mm_P12.70mm_Horizontal"
 			(at 127.762 110.49 90)
 			(hide yes)
@@
 			)
 		)
-		(property "Value" "Q_NPN_BCE"
+		(property "Value" "Q_NPN_CBE"
 			(at 132.08 73.6599 0)
 			(show_name no)
@@
 			)
 		)
-		(property "Footprint" "Package_TO_SOT_THT:TO-92_Inline"
+		(property "Footprint" "Monkey_Riot_Pedals_Library:TO-92L_INLINE_WIDE"
 			(at 132.08 69.85 0)
 			(hide yes)
@@
 			)
 		)
-		(property "Footprint" "Resistor_THT:R_Axial_DIN0207_L6.3mm_D2.5mm_P7.62mm_Horizontal"
+		(property "Footprint" "Resistor_THT:R_Axial_DIN0204_L3.6mm_D1.6mm_P7.62mm_Horizontal"
 			(at 127.762 58.42 90)
 			(hide yes)
@@
 			)
 		)
-		(property "Footprint" "Diode_THT:D_DO-41_SOD81_P10.16mm_Horizontal"
+		(property "Footprint" "Diode_THT:D_DO-41_SOD81_P7.62mm_Horizontal"
 			(at 152.4 102.235 0)
 			(hide yes)
@@
 	(symbol
 		(lib_id "Device:R")
-		(at 125.73 62.23 90)
+		(at 125.73 62.23 270)
 		(unit 1)
 		(body_style 1)
@@
 			)
 		)
-		(property "Footprint" "Resistor_THT:R_Axial_DIN0207_L6.3mm_D2.5mm_P2.54mm_Vertical"
-			(at 125.73 64.008 90)
+		(property "Footprint" "Resistor_THT:R_Axial_DIN0204_L3.6mm_D1.6mm_P2.54mm_Vertical"
+			(at 125.73 60.452 90)
 			(hide yes)
 			(show_name no)
@@
 			)
 		)
-		(property "Footprint" "Diode_THT:D_DO-41_SOD81_P10.16mm_Horizontal"
+		(property "Footprint" "Diode_THT:D_DO-41_SOD81_P7.62mm_Horizontal"
 			(at 152.4 102.235 0)
 			(hide yes)

Commit message: pcb update
Parts:
- R3: footprint Resistor_THT:R_Axial_DIN0309_L9.0mm_D3.2mm_P12.70mm_Horizontal -> Resistor_THT:R_Axial_DIN0207_L6.3mm_D2.5mm_P10.16mm_Horizontal
Changed lines of the file:
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@@
 			)
 		)
-		(property "Footprint" "Resistor_THT:R_Axial_DIN0309_L9.0mm_D3.2mm_P12.70mm_Horizontal"
+		(property "Footprint" "Resistor_THT:R_Axial_DIN0207_L6.3mm_D2.5mm_P10.16mm_Horizontal"
 			(at 127.762 110.49 90)
 			(hide yes)

Commit message: scheme re-design
Parts:
- R2: value R3.3M -> R2.2M
- RV1: value R_Potentiometer -> 5k
- RV2: value R_Potentiometer -> 100k
- RV3: value R_Potentiometer -> 1M
Connections:
- net at J1.T: now also RV2.2; no longer RV3.2
- net at C2.1, Q1.1 (B): now also RV3.1; no longer R2.2
- new net: R2.2, RV3.2
Other:
- moved on the sheet: R2, RV3
Changed lines of the file:
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@@
 	(paper "A4")
-	(junction
-		(at 121.92 66.04)
-		(diameter 0)
-		(color 0 0 0 0)
-	)
 	(junction
 		(at 156.21 83.82)
@@
 	)
 	(junction
+		(at 116.84 66.04)
+		(diameter 0)
+		(color 0 0 0 0)
+	)
+	(junction
 		(at 156.21 106.68)
 		(diameter 0)
@@
 	)
 	(junction
+		(at 107.95 120.65)
+		(diameter 0)
+		(color 0 0 0 0)
+	)
+	(junction
 		(at 148.59 97.79)
 		(diameter 0)
@@
 	(wire
 		(pts
-			(xy 121.92 66.04) (xy 160.02 66.04)
+			(xy 110.49 66.04) (xy 116.84 66.04)
 		)
 		(stroke
@@
 	(wire
 		(pts
-			(xy 111.76 48.26) (xy 149.86 48.26)
-		)
-		(stroke
-			(width 0)
-			(type default)
-		)
-	)
-	(wire
-		(pts
-			(xy 121.92 66.04) (xy 121.92 72.39)
+			(xy 110.49 66.04) (xy 110.49 72.39)
+		)
+		(stroke
+			(width 0)
+			(type default)
+		)
+	)
+	(wire
+		(pts
+			(xy 128.27 62.23) (xy 129.54 62.23)
+		)
+		(stroke
+			(width 0)
+			(type default)
+		)
+	)
+	(wire
+		(pts
+			(xy 110.49 72.39) (xy 121.92 72.39)
+		)
+		(stroke
+			(width 0)
+			(type default)
+		)
+	)
+	(wire
+		(pts
+			(xy 107.95 66.04) (xy 107.95 120.65)
 		)
 		(stroke
@@
 	(wire
 		(pts
+			(xy 107.95 120.65) (xy 129.54 120.65)
+		)
+		(stroke
+			(width 0)
+			(type default)
+		)
+	)
+	(wire
+		(pts
 			(xy 148.59 83.82) (xy 148.59 97.79)
 		)
@@
 	(wire
 		(pts
-			(xy 111.76 35.56) (xy 111.76 40.64)
+			(xy 111.76 62.23) (xy 120.65 62.23)
 		)
 		(stroke
@@
 	(wire
 		(pts
+			(xy 116.84 66.04) (xy 160.02 66.04)
+		)
+		(stroke
+			(width 0)
+			(type default)
+		)
+	)
+	(wire
+		(pts
 			(xy 101.6 91.44) (xy 95.25 91.44)
 		)
@@
 	(wire
 		(pts
-			(xy 99.06 120.65) (xy 129.54 120.65)
+			(xy 107.95 58.42) (xy 116.84 58.42)
+		)
+		(stroke
+			(width 0)
+			(type default)
+		)
+	)
+	(wire
+		(pts
+			(xy 99.06 120.65) (xy 107.95 120.65)
 		)
 		(stroke
@@
 	(wire
 		(pts
+			(xy 116.84 58.42) (xy 116.84 66.04)
+		)
+		(stroke
+			(width 0)
+			(type default)
+		)
+	)
+	(wire
+		(pts
 			(xy 133.35 125.73) (xy 133.35 120.65)
 		)
@@
 	(wire
 		(pts
-			(xy 121.92 62.23) (xy 121.92 66.04)
-		)
-		(stroke
-			(width 0)
-			(type default)
-		)
-	)
-	(wire
-		(pts
 			(xy 156.21 83.82) (xy 156.21 90.17)
 		)
@@
 	(wire
 		(pts
-			(xy 107.95 44.45) (xy 101.6 44.45)
+			(xy 101.6 48.26) (xy 149.86 48.26)
 		)
 		(stroke
@@
 	(wire
 		(pts
-			(xy 101.6 44.45) (xy 101.6 91.44)
+			(xy 101.6 48.26) (xy 101.6 91.44)
 		)
 		(stroke
@@
 			)
 		)
-		(property "Value" "R_Potentiometer"
+		(property "Value" "5k"
 			(at 176.53 67.3099 0)
 			(show_name no)
@@
 			)
 		)
-		(property "Value" "R_Potentiometer"
+		(property "Value" "100k"
 			(at 156.21 49.5299 0)
 			(show_name no)
@@
 				(path "/e5fa3d74-00bc-4c99-a86b-34f1fd700cd0"
 					(reference "RV2")
-					(unit 1)
-				)
-			)
-		)
-	)
-	(symbol
-		(lib_id "power:GND")
-		(at 111.76 35.56 180)
-		(unit 1)
-		(body_style 1)
-		(exclude_from_sim no)
-		(in_bom yes)
-		(on_board yes)
-		(in_pos_files yes)
-		(dnp no)
-		(fields_autoplaced yes)
-		(property "Reference" "#PWR04"
-			(at 111.76 29.21 0)
-			(hide yes)
-			(show_name no)
-			(do_not_autoplace no)
-			(effects
-				(font
-					(size 1.27 1.27)
-				)
-			)
-		)
-		(property "Value" "GND"
-			(at 111.76 30.48 0)
-			(show_name no)
-			(do_not_autoplace no)
-			(effects
-				(font
-					(size 1.27 1.27)
-				)
-			)
-		)
-		(property "Footprint" ""
-			(at 111.76 35.56 0)
-			(hide yes)
-			(show_name no)
-			(do_not_autoplace no)
-			(effects
-				(font
-					(size 1.27 1.27)
-				)
-			)
-		)
-		(property "Datasheet" ""
-			(at 111.76 35.56 0)
-			(hide yes)
-			(show_name no)
-			(do_not_autoplace no)
-			(effects
-				(font
-					(size 1.27 1.27)
-				)
-			)
-		)
-		(property "Description" "Power symbol creates a global label with name \"GND\" , ground"
-			(at 111.76 35.56 0)
-			(hide yes)
-			(show_name no)
-			(do_not_autoplace no)
-			(effects
-				(font
-					(size 1.27 1.27)
-				)
-			)
-		)
-		(pin "1"
-		)
-		(instances
-			(project "electra_000"
-				(path "/e5fa3d74-00bc-4c99-a86b-34f1fd700cd0"
-					(reference "#PWR04")
 					(unit 1)
 				)
@@
 	(symbol
 		(lib_id "Device:R_Potentiometer")
-		(at 111.76 44.45 180)
+		(at 107.95 62.23 0)
 		(unit 1)
 		(body_style 1)
@@
 		(fields_autoplaced yes)
 		(property "Reference" "RV3"
-			(at 114.3 43.1799 0)
+			(at 105.41 60.9599 0)
 			(show_name no)
 			(do_not_autoplace no)
@@
 			)
 		)
-		(property "Value" "R_Potentiometer"
-			(at 114.3 45.7199 0)
+		(property "Value" "1M"
+			(at 105.41 63.4999 0)
 			(show_name no)
 			(do_not_autoplace no)
@@
 		)
 		(property "Footprint" "Monkey_Riot_Pedals_Library:POT_16MM"
-			(at 111.76 44.45 0)
+			(at 107.95 62.23 0)
 			(hide yes)
 			(show_name no)
@@
 		)
 		(property "Datasheet" ""
-			(at 111.76 44.45 0)
+			(at 107.95 62.23 0)
 			(hide yes)
 			(show_name no)
@@
 		)
 		(property "Description" "Potentiometer"
-			(at 111.76 44.45 0)
+			(at 107.95 62.23 0)
 			(hide yes)
 			(show_name no)
@@
 		)
 		(property "Sim.Device" "R"
-			(at 111.76 44.45 0)
+			(at 107.95 62.23 0)
 			(hide yes)
 			(show_name no)
@@
 		)
 		(property "Sim.Type" "POT"
-			(at 111.76 44.45 0)
+			(at 107.95 62.23 0)
 			(hide yes)
 			(show_name no)
@@
 		)
 		(property "Sim.Pins" "1=r0 2=wiper 3=r1"
-			(at 111.76 44.45 0)
+			(at 107.95 62.23 0)
 			(hide yes)
 			(show_name no)
@@
 	(symbol
 		(lib_id "Device:R")
-		(at 125.73 62.23 270)
+		(at 124.46 62.23 270)
 		(unit 1)
 		(body_style 1)
@@
 		(fields_autoplaced yes)
 		(property "Reference" "R2"
-			(at 125.73 55.88 90)
-			(show_name no)
-			(do_not_autoplace no)
-			(effects
-				(font
-					(size 1.27 1.27)
-				)
-			)
-		)
-		(property "Value" "R3.3M"
-			(at 125.73 58.42 90)
+			(at 124.46 55.88 90)
+			(show_name no)
+			(do_not_autoplace no)
+			(effects
+				(font
+					(size 1.27 1.27)
+				)
+			)
+		)
+		(property "Value" "R2.2M"
+			(at 124.46 58.42 90)
 			(show_name no)
 			(do_not_autoplace no)
@@
 		)
 		(property "Footprint" "Resistor_THT:R_Axial_DIN0204_L3.6mm_D1.6mm_P2.54mm_Vertical"
-			(at 125.73 60.452 90)
+			(at 124.46 60.452 90)
 			(hide yes)
 			(show_name no)
@@
 		)
 		(property "Datasheet" ""
-			(at 125.73 62.23 0)
+			(at 124.46 62.23 0)
 			(hide yes)
 			(show_name no)
@@
 		)
 		(property "Description" "Resistor"
-			(at 125.73 62.23 0)
+			(at 124.46 62.23 0)
 			(hide yes)
 			(show_name no)
@@
 		)
 		(property "KiLib_Generator" "resistor/THT"
-			(at 125.73 62.23 0)
-			(hide yes)
-			(show_name no)
+			(at 124.46 62.23 0)
+			(hide yes)
+			(show_name no)
